File: Robotic Arm.kicad_sch (KiCad schematic)
At the start: 1 part

Commit message: try
try
Parts:
- added U?: 4017, symbol 4xxx:4017
Changed lines of the file:
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@@
     (pin "5")
+  )
+  (symbol (lib_id "4xxx:4017") (at 171.45 95.25 0) (unit 1)
+    (in_bom yes) (on_board yes) (fields_autoplaced)
+    (property "Reference" "U?" (id 0) (at 173.4694 74.93 0)
+      (effects (font (size 1.27 1.27)) (justify left))
+    )
+    (property "Value" "4017" (id 1) (at 173.4694 77.47 0)
+      (effects (font (size 1.27 1.27)) (justify left))
+    )
+    (property "Footprint" "" (id 2) (at 171.45 95.25 0)
+      (effects (font (size 1.27 1.27)) hide)
+    )
+    (property "Datasheet" "http://www.intersil.com/content/dam/Intersil/documents/cd40/cd4017bms-22bms.pdf" (id 3) (at 171.45 95.25 0)
+      (effects (font (size 1.27 1.27)) hide)
+    )
+    (pin "1")
+    (pin "10")
+    (pin "11")
+    (pin "12")
+    (pin "13")
+    (pin "14")
+    (pin "15")
+    (pin "16")
+    (pin "2")
+    (pin "3")
+    (pin "4")
+    (pin "5")
+    (pin "6")
+    (pin "7")
+    (pin "8")
+    (pin "9")
   )
   (sheet_instances
@@
       (reference "U?") (unit 1) (value "74AHC1G86") (footprint "")
     )
+    (path "/da9fdfe2-960c-4634-ab46-2284dfe404c2"
+      (reference "U?") (unit 1) (value "4017") (footprint "")
+    )
   )

Commit message: Inital system setup
Parts:
- removed U?: 74AHC1G86, symbol 74xGxx:74AHC1G86
- removed U?: 4017, symbol 4xxx:4017
- added A?: Pololu_Breakout_DRV8825, Module:Pololu_Breakout-16_15.2x20.3mm, symbol Driver_Motor:Pololu_Breakout_DRV8825
- added J? (x2): Conn_01x20_Female, symbol Connector:Conn_01x20_Female
- added M?: Stepper_Motor_bipolar, symbol Motor:Stepper_Motor_bipolar
Changed lines of the file:
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@@
 (kicad_sch (version 20211123) (generator eeschema)
   (paper "A4")
-  (symbol (lib_id "74xGxx:74AHC1G86") (at 123.19 88.9 0) (unit 1)
+  (symbol (lib_id "Driver_Motor:Pololu_Breakout_DRV8825") (at 160.02 80.01 0) (unit 1)
     (in_bom yes) (on_board yes) (fields_autoplaced)
-    (property "Reference" "U?" (id 0) (at 122.2375 81.28 0))
-    (property "Value" "74AHC1G86" (id 1) (at 122.2375 83.82 0))
-    (property "Footprint" "" (id 2) (at 123.19 88.9 0)
-      (effects (font (size 1.27 1.27)) hide)
-    )
-    (property "Datasheet" "http://www.ti.com/lit/sg/scyt129e/scyt129e.pdf" (id 3) (at 123.19 88.9 0)
-      (effects (font (size 1.27 1.27)) hide)
-    )
-    (pin "1")
-    (pin "2")
-    (pin "3")
-    (pin "4")
-    (pin "5")
-  )
-  (symbol (lib_id "4xxx:4017") (at 171.45 95.25 0) (unit 1)
-    (in_bom yes) (on_board yes) (fields_autoplaced)
-    (property "Reference" "U?" (id 0) (at 173.4694 74.93 0)
+    (property "Reference" "A?" (id 0) (at 162.0394 62.23 0)
       (effects (font (size 1.27 1.27)) (justify left))
     )
-    (property "Value" "4017" (id 1) (at 173.4694 77.47 0)
+    (property "Value" "Pololu_Breakout_DRV8825" (id 1) (at 162.0394 64.77 0)
       (effects (font (size 1.27 1.27)) (justify left))
     )
-    (property "Footprint" "" (id 2) (at 171.45 95.25 0)
-      (effects (font (size 1.27 1.27)) hide)
+    (property "Footprint" "Module:Pololu_Breakout-16_15.2x20.3mm" (id 2) (at 165.1 100.33 0)
+      (effects (font (size 1.27 1.27)) (justify left) hide)
     )
-    (property "Datasheet" "http://www.intersil.com/content/dam/Intersil/documents/cd40/cd4017bms-22bms.pdf" (id 3) (at 171.45 95.25 0)
+    (property "Datasheet" "https://www.pololu.com/product/2982" (id 3) (at 162.56 87.63 0)
       (effects (font (size 1.27 1.27)) hide)
     )
@@
     (pin "9")
   )
+  (symbol (lib_id "Motor:Stepper_Motor_bipolar") (at 203.2 83.82 0) (unit 1)
+    (in_bom yes) (on_board yes) (fields_autoplaced)
+    (property "Reference" "M?" (id 0) (at 208.28 81.699 0)
+      (effects (font (size 1.27 1.27)) (justify left))
+    )
+    (property "Value" "Stepper_Motor_bipolar" (id 1) (at 208.28 84.239 0)
+      (effects (font (size 1.27 1.27)) (justify left))
+    )
+    (property "Footprint" "" (id 2) (at 203.454 84.074 0)
+      (effects (font (size 1.27 1.27)) hide)
+    )
+    (property "Datasheet" "http://www.infineon.com/dgdl/Application-Note-TLE8110EE_driving_UniPolarStepperMotor_V1.1.pdf?fileId=db3a30431be39b97011be5d0aa0a00b0" (id 3) (at 203.454 84.074 0)
+      (effects (font (size 1.27 1.27)) hide)
+    )
+    (pin "1")
+    (pin "2")
+    (pin "3")
+    (pin "4")
+  )
+  (symbol (lib_id "Connector:Conn_01x20_Female") (at 119.38 78.74 0) (unit 1)
+    (in_bom yes) (on_board yes)
+    (property "Reference" "J?" (id 0) (at 120.65 78.7399 0)
+      (effects (font (size 1.27 1.27)) (justify left))
+    )
+    (property "Value" "Conn_01x20_Female" (id 1) (at 120.65 100.33 90)
+      (effects (font (size 1.27 1.27)) (justify left))
+    )
+    (property "Footprint" "" (id 2) (at 119.38 78.74 0)
+      (effects (font (size 1.27 1.27)) hide)
+    )
+    (property "Datasheet" "~" (id 3) (at 119.38 78.74 0)
+      (effects (font (size 1.27 1.27)) hide)
+    )
+    (pin "1")
+    (pin "10")
+    (pin "11")
+    (pin "12")
+    (pin "13")
+    (pin "14")
+    (pin "15")
+    (pin "16")
+    (pin "17")
+    (pin "18")
+    (pin "19")
+    (pin "2")
+    (pin "20")
+    (pin "3")
+    (pin "4")
+    (pin "5")
+    (pin "6")
+    (pin "7")
+    (pin "8")
+    (pin "9")
+  )
+  (symbol (lib_id "Connector:Conn_01x20_Female") (at 130.81 81.28 180) (unit 1)
+    (in_bom yes) (on_board yes)
+    (property "Reference" "J?" (id 0) (at 129.54 78.74 0))
+    (property "Value" "Conn_01x20_Female" (id 1) (at 129.54 91.44 90))
+    (property "Footprint" "" (id 2) (at 130.81 81.28 0)
+      (effects (font (size 1.27 1.27)) hide)
+    )
+    (property "Datasheet" "~" (id 3) (at 130.81 81.28 0)
+      (effects (font (size 1.27 1.27)) hide)
+    )
+    (pin "1")
+    (pin "10")
+    (pin "11")
+    (pin "12")
+    (pin "13")
+    (pin "14")
+    (pin "15")
+    (pin "16")
+    (pin "17")
+    (pin "18")
+    (pin "19")
+    (pin "2")
+    (pin "20")
+    (pin "3")
+    (pin "4")
+    (pin "5")
+    (pin "6")
+    (pin "7")
+    (pin "8")
+    (pin "9")
+  )
   (sheet_instances
     (path "/" (page "1"))
   )
   (symbol_instances
-    (path "/b19fa3d8-cad3-44b7-8500-f61d8b27a60b"
-      (reference "U?") (unit 1) (value "74AHC1G86") (footprint "")
+    (path "/2cdaab39-81f1-4593-98a9-4b3ba5375c9d"
+      (reference "A?") (unit 1) (value "Pololu_Breakout_DRV8825") (footprint "Module:Pololu_Breakout-16_15.2x20.3mm")
     )
-    (path "/da9fdfe2-960c-4634-ab46-2284dfe404c2"
-      (reference "U?") (unit 1) (value "4017") (footprint "")
+    (path "/88f34814-d19d-475f-b6f3-250cfa44cf4a"
+      (reference "J?") (unit 1) (value "Conn_01x20_Female") (footprint "")
+    )
+    (path "/c894312a-55df-4d9f-9528-7bb742c76d1d"
+      (reference "J?") (unit 1) (value "Conn_01x20_Female") (footprint "")
+    )
+    (path "/419136ec-6193-4acf-90cb-5e351c718bae"
+      (reference "M?") (unit 1) (value "Stepper_Motor_bipolar") (footprint "")
     )
   )

Commit message: ch
Connections:
- net at A?.4 (A1): now also M?.1
Changed lines of the file:
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@@
 (kicad_sch (version 20211123) (generator eeschema)
   (paper "A4")
+  (wire (pts (xy 170.18 76.2) (xy 170.18 77.47))
+    (stroke (width 0) (type default) (color 0 0 0 0))
+  )
+  (wire (pts (xy 200.66 76.2) (xy 170.18 76.2))
+    (stroke (width 0) (type default) (color 0 0 0 0))
+  )
   (symbol (lib_id "Driver_Motor:Pololu_Breakout_DRV8825") (at 160.02 80.01 0) (unit 1)
     (in_bom yes) (on_board yes) (fields_autoplaced)
